File: electronics/TinXsat/_autosave-TinXsat.sch (KiCad schematic (older format))
At the start: 67 parts

Commit message: pcb update (not finished yet)
Parts:
- removed C?: 470n, Capacitor_SMD:C_0805_2012Metric_Pad1.18x1.45mm_HandSolder, symbol Device:C
- removed C?: 22uF/10V, Capacitor_SMD:C_1210_3225Metric_Pad1.33x2.70mm_HandSolder, symbol Device:C
- removed D? (x2): SMS240, Diode_SMD:D_MELF, symbol Diode:1N5711UR
- removed D? (x2): 5.1V, symbol Device:D_Zener
- removed L?: 4.7uH/2.9A, Inductor_SMD:L_7.3x7.3_H3.5, symbol Device:L
- removed Q?: IRF7406, Package_SO:SOIC-8_3.9x4.9mm_P1.27mm, symbol Transistor_FET:IRF7404
- removed R?: 100m, Resistor_SMD:R_MiniMELF_MMA-0204, symbol Device:R
- removed R?: 2k2, Resistor_SMD:R_0805_2012Metric_Pad1.20x1.40mm_HandSolder, symbol Device:R
- removed R?: 390k, Resistor_SMD:R_0805_2012Metric_Pad1.20x1.40mm_HandSolder, symbol Device:R
- removed U?: LTC4002ES8-4.2, Package_SO:SOIC-8_3.9x4.9mm_P1.27mm, symbol Battery_Management:LTC4002ES8-4.2
- added BZ1: Buzzer, Zasilacz_brama:PinHeader_1x02_P2.54mm_SMD, symbol Device:Buzzer
- added C11: 2n2, Capacitor_SMD:C_0805_2012Metric_Pad1.18x1.45mm_HandSolder, symbol Device:C
- added C13, C15, C20: 22u, Capacitor_SMD:C_1210_3225Metric_Pad1.33x2.70mm_HandSolder, symbol Device:C
- added C14, C18, C19, C2, C22, C27, C3, C30, C33, C35, C37, C38, C39, C4, C40, C41, C42, C43, C46, C47, C7, C9: 100n, Capacitor_SMD:C_0805_2012Metric_Pad1.18x1.45mm_HandSolder, symbol Device:C
- added C23, C32, C5: 22uF/10V, Capacitor_SMD:C_1210_3225Metric_Pad1.33x2.70mm_HandSolder, symbol Device:C
- added C25, C28: 20p, Capacitor_SMD:C_0603_1608Metric_Pad1.08x0.95mm_HandSolder, symbol Device:C
- added C26, C29: 6p8, Capacitor_SMD:C_0603_1608Metric_Pad1.08x0.95mm_HandSolder, symbol Device:C
- added C45, C8: 10u, Capacitor_SMD:C_1206_3216Metric_Pad1.33x1.80mm_HandSolder, symbol Device:C
- added D1: GREEN, LED_SMD:LED_0805_2012Metric_Pad1.15x1.40mm_HandSolder, symbol Device:LED
- added D2: BLUE, LED_SMD:LED_0805_2012Metric_Pad1.15x1.40mm_HandSolder, symbol Device:LED
- added D3, D9: SMS240, Diode_SMD:D_MELF, symbol Diode:1N5711UR
- added D4: LED_RGCB, Zasilacz_brama:LED_D5.0mm-4_RGB, symbol Device:LED_RGCB
- added D6: TXDIODE, LED_SMD:LED_0805_2012Metric_Pad1.15x1.40mm_HandSolder, symbol Device:LED
- added D7: RXDIODE, LED_SMD:LED_0805_2012Metric_Pad1.15x1.40mm_HandSolder, symbol Device:LED
- added J10: CAN, Zasilacz_brama:PinHeader_1x03_P2.00mm_SMD, symbol Connector:Conn_01x03_Female
- added J2: ESP-PROG, Zasilacz_brama:PinHeader_1x05_P2.54mm_SMD, symbol Connector:Conn_01x05_Female
- added J3: POWER_LED, Zasilacz_brama:PinHeader_1x05_P2.54mm_SMD, symbol Connector:Conn_01x05_Female
- added J4: MCO_OUT, Connector_PinHeader_2.54mm:PinHeader_1x01_P2.54mm_Vertical, symbol Connector:Conn_01x01_Male
- added J5: BMP280_1, Zasilacz_brama:PinHeader_1x06_P2.00mm_SMD, symbol Connector:Conn_01x06_Female
- added J6: BMP280_2, Zasilacz_brama:PinHeader_1x06_P2.00mm_SMD, symbol Connector:Conn_01x06_Female
- added J7: ESP-card, Zasilacz_brama:PinHeader_1x08_P2.00mm_SMD, symbol Connector:Conn_01x09_Female
- added J8: GPS, Zasilacz_brama:PinHeader_1x04_P2.54mm_SMD, symbol Connector:Conn_01x04_Female
- added J9: SWD, Zasilacz_brama:PinHeader_1x06_P2.00mm_SMD, symbol Connector:Conn_01x06_Female
- added L2: 22uH/3A, Inductor_SMD:L_7.3x7.3_H3.5, symbol Device:L
- added L3: BEAD, Inductor_SMD:L_0805_2012Metric_Pad1.05x1.20mm_HandSolder, symbol Device:L
- added Q7: BSS138, Package_TO_SOT_SMD:SOT-23, symbol Transistor_FET:BSS138
- added Q8: STD7NK40Z, Package_TO_SOT_SMD:TO-252-2, symbol Transistor_FET:STD7NK40Z
- added R1, R14, R15, R16, R25, R31, R33, R34, R35, R45, R46, R47, R48: 10k, Resistor_SMD:R_0805_2012Metric_Pad1.20x1.40mm_HandSolder, symbol Device:R
- added R11, R18: 470, Resistor_SMD:R_0805_2012Metric_Pad1.20x1.40mm_HandSolder, symbol Device:R
- added R2, R4, R56, R57, R58: 47, Resistor_SMD:R_0805_2012Metric_Pad1.20x1.40mm_HandSolder, symbol Device:R
- added R27, R52, R53: 2k2, Resistor_SMD:R_0805_2012Metric_Pad1.20x1.40mm_HandSolder, symbol Device:R
- added R3, R44: 1k, Resistor_SMD:R_0805_2012Metric_Pad1.20x1.40mm_HandSolder, symbol Device:R
- added R32: 22m, Resistor_SMD:R_MiniMELF_MMA-0204, symbol Device:R
- added R36, R39: 390, Resistor_SMD:R_0805_2012Metric_Pad1.20x1.40mm_HandSolder, symbol Device:R
- added R37, R40, R60: 0, Resistor_SMD:R_0805_2012Metric_Pad1.20x1.40mm_HandSolder, symbol Device:R
- added R42, R43: R, Resistor_SMD:R_0805_2012Metric_Pad1.20x1.40mm_HandSolder, symbol Device:R
- added U1: CP2102N-A01-GQFN28, Package_DFN_QFN:QFN-28-1EP_5x5mm_P0.5mm_EP3.35x3.35mm, symbol Interface_USB:CP2102N-A01-GQFN28
- added U10: TPS61175PWP, footprints:TPS61175PWP, symbol 2020-12-09_12-36-17:TPS61175PWP
- added U11: STM32F103RGTx, Package_QFP:LQFP-64_10x10mm_P0.5mm, symbol MCU_ST_STM32F1:STM32F103RGTx
- added U12, U13, U14: LM35-LP, Zasilacz_brama:PinHeader_1x03_P2.00mm_SMD, symbol Sensor_Temperature:LM35-LP
- added U2: A25L032, Package_SO:SOP-8_3.9x4.9mm_P1.27mm, symbol sch-lib:A25L032
- added U3: MPU-6050, Sensor_Motion:InvenSense_QFN-24_4x4mm_P0.5mm, symbol Sensor_Motion:MPU-6050
- added U4: TP4056, Package_SO:SOIC-8-1EP_3.9x4.9mm_P1.27mm_EP2.29x3mm, symbol tp4056:TP4056
- added U5: Ai-Thinker-Ra-01, RF_Module:Ai-Thinker-Ra-01-LoRa, symbol RF_Module:Ai-Thinker-Ra-01
- added U6: ESP32-cam, Zasilacz_brama:ESP32-CAM, symbol sch-lib:ESP32-cam
- added U7: INA219AxDCN, Package_TO_SOT_SMD:SOT-23-8, symbol Analog_ADC:INA219AxDCN
- added U8: MCP130, Package_TO_SOT_SMD:SOT-23, symbol Power_Supervisor:MCP130-xxxxTT
- added XS1: SD_ebay-uSD-push_push_SMD, footprints:Conn_uSDcard, symbol uSD_push-push_ebay:SD_ebay-uSD-push_push_SMD
- added Y1: 8Mhz, Crystal:Crystal_SMD_HC49-SD, symbol Device:Crystal
- added Y2: 32768Hz, Crystal:Crystal_DS26_D2.0mm_L6.0mm_Horizontal_1EP_style1, symbol Device:Crystal
- BT1, BT2: renamed from BT?; footprint (none) -> Zasilacz_brama:BATT
- C17, C24, C34: renamed from C?; value 22uF/10V -> 10uF/10V; footprint Capacitor_SMD:C_1210_3225Metric_Pad1.33x2.70mm_HandSolder -> Capacitor_SMD:C_1206_3216Metric_Pad1.33x1.80mm_HandSolder
- F1, F2, F3: renamed from F?; footprint (none) -> Fuse:Fuse_1206_3216Metric_Pad1.42x1.75mm_HandSolder
- J1: renamed from J?; footprint (none) -> Connector_USB:USB_Mini-B_Lumberg_2486_01_Horizontal
- R10, R12, R13, R17, R19, R20, R21, R22, R23, R26, R29, R30, R5, R6, R7, R8, R9: renamed from R?; footprint (none) -> Resistor_SMD:R_0805_2012Metric_Pad1.20x1.40mm_HandSolder
- R38, R59: renamed from R?; footprint Resistor_SMD:R_MiniMELF_MMA-0204 -> Resistor_SMD:R_0805_2012Metric_Pad1.20x1.40mm_HandSolder
- SW1: renamed from SW?; footprint (none) -> Button_Switch_THT:SW_Tactile_SKHH_Angled
- TH1: renamed from TH?; footprint (none) -> Zasilacz_brama:PinHeader_1x02_P2.54mm_SMD
- gave numbers to parts that had none: 25
Connections:
- net +3V3: now also C31.2, U9.4 (VS), C13.2, C14.2, C15.2, C18.2, C19.1, C20.2, C22.2, C3.2, C30.1, C35.1, C37.1, C38.1, C39.2, C4.2, C40.2, C41.2, C42.2, C43.1, C45.1, C46.1, C7.1, C8.2, J2.2 (Pin_2), J3.1 (Pin_1), J5.1 (Pin_1), J6.1 (Pin_1), J6.6 (Pin_6), J8.1 (Pin_1), J9.1 (Pin_1), L3.1, R11.1, R15.2, R18.1, R33.1, R52.2, R53.1, U1.6 (VDD), U11.19 (VDD), U11.32 (VDD), U11.48 (VDD), U11.64 (VDD), U12.1 (+VS), U13.1 (+VS), U14.1 (+VS), U2.8 (VCC), U3.13 (VDD), U3.8 (VDDIO), U5.3 (3v3), U6.16 (3V3), U7.4 (VS), U8.2 (VDD)
- net CHRG_READ: now also R25.1, U11.21 (PA5); no longer R24.1
- net CHRH_PULL: now also U11.20 (PA4)
- net GND: now also C11.1, C13.1, C14.1, C15.1, C18.1, C19.2, C2.2, C20.1, C22.1, C23.2, C25.2, C26.2, C27.1, C28.2, C29.2, C3.1, C30.2, C32.2, C33.2, C35.2, C37.2, C38.2, C39.1, C4.1, C40.1, C41.1, C42.1, C43.2, C45.2, C46.2, C47.2, C5.2, C7.2, C8.1, C9.1, D1.1 (K), D2.1 (K), D4.3 (K), J10.3 (Pin_3), J2.5 (Pin_5), J3.3 (Pin_3), J5.2 (Pin_2), J5.6 (Pin_6), J6.2 (Pin_2), J7.6 (Pin_6), J8.4 (Pin_4), J9.3 (Pin_3), Q7.2 (S), Q8.3 (S), R14.1, R16.2, R27.2, R31.1, R34.1, R43.1, R45.1, R47.1, R48.2, U1.29 (GND), U1.3 (GND), U10.12 (PGND), U10.13 (PGND), U10.14 (PGND), U10.15 (EPAD), U10.6 (SYNC), U10.7 (AGND), U11.12 (VSSA), U11.18 (VSS), U11.31 (VSS), U11.47 (VSS), U11.60 (BOOT0), U11.63 (VSS), U12.3 (GND), U13.3 (GND), U14.3 (GND), U2.4 (VSS), U3.18 (GND), U4.3 (GND), U4.9 (PP), U5.16 (Gnd), U5.2 (Gnd), U5.9 (Gnd), U6.13 (GND), U6.2 (GND), U6.9 (GND), U7.3 (GND), U7.7 (A0), U7.8 (A1), U8.3 (VSS), XS1.6 (GND)
- net PWR_BUTTON: now also U11.14 (PA0)
- net PWR_KEEP: now also U11.2 (PC13)
- net STM_USBDM: now also J10.1 (Pin_1), U11.44 (PA11)
- net STM_USBDP: now also J10.2 (Pin_2), U11.45 (PA12)
- net UART_DM: now also U1.5 (D-)
- net UART_DP: now also U1.4 (D+)
- net VBUS: now also C2.1, D3.1 (K), U1.7 (REGIN), U1.8 (VBUS), U4.4 (VCC); no longer F1.1, R29.2
- net VBUS_ADC: now also U11.15 (PA1)
- net at C24.1, R38.1, R41.2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: now also U4.5 (BAT)
- net at R28.2, TH1.1: now also U4.1 (TEMP)
- net at D10.1 (K), F2.2, F3.2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: now also R60.1
- net SYSTEM_SCL: now reaches U9.5 (SCL)
- net SYSTEM_SCL: now also J5.3 (Pin_3), J6.3 (Pin_3), R52.1, U11.58 (PB6), U7.5 (SCL)
- net SYSTEM_SDA: now reaches U9.6 (SDA)
- net SYSTEM_SDA: now also J5.4 (Pin_4), J6.4 (Pin_4), R53.2, U11.59 (PB7), U7.6 (SDA)
- new net: C33.1, L3.2, U11.13 (VDDA)
- new net: R37.1, U11.3 (PC14)
- new net: R40.1, U11.4 (PC15)
- new net: J4.1 (Pin_1), U11.41 (PA8)
- new net: R36.1, U11.5 (PD0)
- new net: R39.1, U11.6 (PD1)
- new net: R24.1, U4.8 (CE)
- new net: D4.4 (BA), R56.1
- new net: D4.2 (GA), R57.1
- new net: D4.1 (RA), R58.1
- new net: J2.1 (Pin_1), U6.14 (GPIO0)
- new net: R31.2, U6.5 (GPIO15)
- new net: D1.2 (A), R2.1
- new net: D2.2 (A), R4.1
- new net: J7.1 (Pin_1), XS1.1 (DAT2)
- new net: J7.2 (Pin_2), XS1.2 (CS/DAT3)
- new net: J7.3 (Pin_3), XS1.3 (DI/CMD)
- new net: J7.4 (Pin_4), XS1.4 (Vdd)
- new net: J7.5 (Pin_5), XS1.5 (CLK)
- new net: J7.7 (Pin_7), XS1.7 (DO/DAT0)
- new net: J7.8 (Pin_8), XS1.8 (DAT1)
- new net: J7.9 (Pin_9), XS1.9 (CD)
- new net: BZ1.2 (+), Q7.3 (D)
- new net: Q7.1 (G), R3.1, R34.2
- new net: R27.1, U4.2 (PROG)
- new net: R25.2, U4.6 (~STDBY)
- new net: R15.1, U2.7 (NC)
- new net: Q8.1 (G), R44.1, R45.2
- new net: J3.5 (Pin_5), Q8.2 (D)
- new net: C25.1, R36.2, Y1.1
- new net: C28.1, R39.2, Y1.2
- new net: C26.1, R37.2, Y2.1
- new net: C29.1, R40.2, Y2.2
- new net: C23.1, C5.1, L2.1, R32.2, U10.3 (VIN), U7.2 (IN-)
- new net: R16.1, U3.1 (CLKIN)
- new net: C11.2, C9.2, U3.10 (REGOUT)
- new net: R14.2, U3.9 (AD0)
- new net: D7.1 (K), U1.18 (~RXT~/GPIO.1)
- new net: D6.1 (K), U1.19 (~TXT~/GPIO.0)
- new net: R1.1, U1.9 (~RSTb)
- new net: D6.2 (A), R11.2
- new net: D7.2 (A), R18.2
- new net: R35.2, U10.4 (EN)
- new net: D9.2 (A), L2.2, U10.1 (SW), U10.2 (SW)
- new net: R46.2, U10.10 (FREQ)
- new net: C27.2, U10.5 (SS)
- new net: R42.1, R43.2, U10.9 (FB)
- new net: R46.1, R47.2, R48.1
- new net +3.3VP: R1.2
- new net +VSW: BZ1.1 (-), C32.1, D9.1 (K), J3.4 (Pin_4), R42.2
- new net BAT_TEMP: U11.9 (PC1), U13.2 (Vout)
- new net BUZZER: R3.2, U11.54 (PD2)
- new net CAM-BSY: U11.57 (PB5), U6.3 (GPIO12)
- new net CAM-STROBE: U11.56 (PB4), U6.4 (GPIO13)
- new net DEBUG_LED_1: R4.2, U11.40 (PC9)
- new net DEBUG_LED_2: R2.2, U11.39 (PC8)
- new net DEBUG_RX: U1.26 (TXD), U11.43 (PA10)
- new net DEBUG_TX: U1.25 (RXD), U11.42 (PA9)
- new net ESP-RX: J2.4 (Pin_4), U11.16 (PA2), U6.11 (GPIO3)
- new net ESP-TX: J2.3 (Pin_3), U11.17 (PA3), U6.10 (GPIO1)
- new net ETEMP_1: U11.10 (PC2), U12.2 (Vout)
- new net ETEMP_2: U11.11 (PC3), U14.2 (Vout)
- new net FLASH_CS: U11.33 (PB12), U2.1 (~CS)
- new net FLASH_WP: U11.53 (PC12), U2.3 (~WP~)
- new net GPS_RX: J8.3 (Pin_3), U11.52 (PC11)
- new net GPS_TX: J8.2 (Pin_2), U11.51 (PC10)
- new net GYRO_FRAME: U11.25 (PC5), U3.11 (FSYNC)
- new net GYRO_IRQ: U11.27 (PB1), U3.12 (INT)
- new net GYRO_SCL: U11.29 (PB10), U3.23 (SCL)
- new net GYRO_SDA: U11.30 (PB11), U3.24 (SDA)
- new net LED_TEMP: J3.2 (Pin_2), U11.8 (PC0)
- new net LORA_CS: U11.37 (PC6), U5.15 (~SS)
- new net LORA_IRQ: U11.28 (PB2), U5.5 (DIO0)
- new net LORA_RST: U11.38 (PC7), U5.4 (~Reset)
- new net NRST: C47.1, J9.5 (Pin_5), R33.2, U11.7 (NRST), U8.1 (~RST)
- new net PWR_LED_DIMM: R44.2, U11.62 (PB9)
- new net PWR_LED_ON: R35.1, U11.61 (PB8)
- new net SPI_MISO: U11.35 (PB14), U2.2 (O1/SO), U5.13 (MISO)
- new net SPI_MOSI: U11.36 (PB15), U2.5 (SI/IO0), U5.14 (MOSI)
- new net SPI_SCK: U11.34 (PB13), U2.6 (SCLK), U5.12 (SCK)
- new net STATUS_LED_1: R56.2, U11.22 (PA6)
- new net STATUS_LED_2: R57.2, U11.23 (PA7)
- new net STATUS_LED_3: R58.2, U11.26 (PB0)
- new net SWDCLK: J9.2 (Pin_2), U11.49 (PA14)
- new net SWDIO: J9.4 (Pin_4), U11.46 (PA13)
- new net SWO: J9.6 (Pin_6), U11.55 (PB3)
- new net USB_DET: D3.2 (A), F1.1, R29.2
- new net VD: R32.1, R60.2, U7.1 (IN+)
- no-connect marks 0 -> 8
Other:
- note added: "3V3 SMPS"
- note added: "ADDR = 0x76\n"
- note added: "ADDR = 0x77\n\n"
- note added: "EDGE CONN"
- note added: "ESP-CAM\n"
- note added: "FLASH\n"
- note added: "GYRO"
- note added: "HSE"
- note added: "LORA"
- note added: "PWRLED DRIVER"
- note added: "PWRON LOGIC"
- note added: "SENSORS"
- note added: "STM32"
- note added: "USB & CHARGING"
- note added: "USB/UART BRIDGE"
- note added: "USB_DM = CANRX\nUSB_DP = CANTX"
- note removed: "Rsh=100mV/1A=0,01Ohm"
- moved on the sheet: BT1, BT2, C1, C12, C16, C17, C24, C31, C34, C36, C44, C6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
