File: electronics/TinXsat/TinXsat.kicad_pcb (KiCad board)
At the start: 2 copper layers, 50 x 80 mm, 163 parts, among them J1 USB_B_Mini, J10 CAN, J2 ESP-PROG, J3 POWER_LED, J4 MCO_OUT, J5 BMP280_1, J6 BMP280_2, J7 Micro_SD_Card, J8 GPS, J9 SWD, Q1 Si2371, Q2 Si2371, Q3 BSS138, Q4 BSS138, Q5 Si2371, Q6 BSS138, Q7 IRF7406, Q8 STD7NK40Z, SW1 SW_Push, U1 CP2102N-A01-GQFN28, U10 TPS61175PWP, U11 STM32F103RGTx, U12 LM35-LP, U13 LM35-LP, U14 LM35-LP, U15 TPS63001, U2 A25L032, U3 MPU-6050, U4 LTC4002ES8-4.2, U5 Ai-Thinker-Ra-01, U6 ESP32-cam, U7 INA219AxDCN, U8 MCP130, U9 INA219AxDCN, Y1 8Mhz, Y2 32768Hz

Commit message: pcb initial commit
Parts:
- removed C10: 470n, Capacitor_SMD:C_0805_2012Metric_Pad1.18x1.45mm_HandSolder
- removed C21: 22uF/10V, Capacitor_SMD:C_1210_3225Metric_Pad1.33x2.70mm_HandSolder
- removed D11: 1N4148, Diode_SMD:D_MiniMELF_Handsoldering
- removed D4, D5: 4V7, Diode_SMD:D_MiniMELF_Handsoldering
- removed D8: SMS240, Diode_SMD:D_MELF
- removed L1: 4.7uH/2.9A, Inductor_SMD:L_7.3x7.3_H3.5
- removed Q7: IRF7406, Package_SO:SOIC-8_3.9x4.9mm_P1.27mm
- removed R3: 10k, Resistor_SMD:R_0805_2012Metric_Pad1.20x1.40mm_HandSolder
- removed R34: 100m, Resistor_SMD:R_MiniMELF_MMA-0204
- added XS1: SD_ebay-uSD-push_push_SMD, footprints:Conn_uSDcard, B.Cu at (54.5, 86.6)
- BT1, C18, C19, C20, C22, C25, C26, C28, C29, C30, C46, C47, C6, D1, D2, D6, D7, Q2, Q3, Q5, R17, R19, R2, R22, R23, R24, R26, R31, R33, R4, R42, R43, R46, R47, R48, R52, R53, R9, U8: moved to B.Cu
- C16, C36, D10, R49, R50, R51: moved to F.Cu
- C17: value 22uF/10V -> 10uF/10V; footprint Capacitor_SMD:C_1210_3225Metric_Pad1.33x2.70mm_HandSolder -> Capacitor_SMD:C_1206_3216Metric_Pad1.33x1.80mm_HandSolder; moved to F.Cu
- C24, C34: value 22uF/10V -> 10uF/10V; footprint Capacitor_SMD:C_1210_3225Metric_Pad1.33x2.70mm_HandSolder -> Capacitor_SMD:C_1206_3216Metric_Pad1.33x1.80mm_HandSolder
- C45: value 22u -> 10u; footprint Capacitor_SMD:C_1210_3225Metric_Pad1.33x2.70mm_HandSolder -> Capacitor_SMD:C_1206_3216Metric_Pad1.33x1.80mm_HandSolder; moved to B.Cu
- C8: value 22u -> 10u; footprint Capacitor_SMD:C_1210_3225Metric_Pad1.33x2.70mm_HandSolder -> Capacitor_SMD:C_1206_3216Metric_Pad1.33x1.80mm_HandSolder
- J10: footprint Connector_PinHeader_2.54mm:PinHeader_1x03_P2.54mm_Vertical -> Zasilacz_brama:PinHeader_1x03_P2.00mm_SMD; moved to B.Cu
- J2: footprint Connector_PinHeader_2.54mm:PinHeader_1x05_P2.54mm_Vertical -> Zasilacz_brama:PinHeader_1x05_P2.54mm_SMD; moved to B.Cu
- J3: footprint Connector_PinHeader_2.54mm:PinHeader_1x05_P2.54mm_Vertical -> Zasilacz_brama:PinHeader_1x05_P2.54mm_SMD
- J5, J6: footprint Connector_PinHeader_2.54mm:PinHeader_1x06_P2.54mm_Vertical -> Zasilacz_brama:PinHeader_1x06_P2.00mm_SMD
- J7: value Micro_SD_Card -> ESP-card; footprint Connector_Card:microSD_HC_Molex_104031-0811 -> Zasilacz_brama:PinHeader_1x08_P2.00mm_SMD
- J8: footprint Connector_PinHeader_2.54mm:PinHeader_1x04_P2.54mm_Vertical -> Zasilacz_brama:PinHeader_1x04_P2.54mm_SMD
- J9: footprint Connector_PinHeader_2.54mm:PinHeader_1x06_P2.54mm_Vertical -> Zasilacz_brama:PinHeader_1x06_P2.00mm_SMD; moved to B.Cu
- R25: value 390k -> 10k; moved to B.Cu
- R59: footprint Resistor_SMD:R_MiniMELF_MMA-0204 -> Resistor_SMD:R_0805_2012Metric_Pad1.20x1.40mm_HandSolder
- SW1: footprint Zasilacz_brama:Panasonic_EVQPUK_EVQPUB -> Button_Switch_THT:SW_Tactile_SKHH_Angled
- TH1: footprint Connector_PinHeader_2.54mm:PinHeader_1x02_P2.54mm_Vertical -> Zasilacz_brama:PinHeader_1x02_P2.54mm_SMD; moved to B.Cu
- U10: footprint Package_SO:HTSSOP-14-1EP_4.4x5mm_P0.65mm_EP3.4x5mm_Mask3x3.1mm_ThermalVias -> footprints:TPS61175PWP
- U12, U13, U14: footprint Package_TO_SOT_THT:TO-92 -> Zasilacz_brama:PinHeader_1x03_P2.00mm_SMD
- U4: value LTC4002ES8-4.2 -> TP4056; footprint Package_SO:SOIC-8_3.9x4.9mm_P1.27mm -> Package_SO:SOIC-8-1EP_3.9x4.9mm_P1.27mm_EP2.29x3mm; moved to F.Cu
- Y1: footprint Crystal:Crystal_HC49-U_Vertical -> Crystal:Crystal_SMD_HC49-SD
- moved C25 179.7 mm to (91.1, 85.6), turned to 90 degrees
- moved C26 175.4 mm to (98.3, 95.7), turned to 270 degrees
- moved C29 166.6 mm to (96.4, 95.6), turned to 270 degrees
- moved U13 149.8 mm to (69.3, 128.3), turned to 270 degrees
- moved D9 148.9 mm to (61.6, 58.5), turned to 270 degrees
- moved C30 148.7 mm to (88.6, 90.0)
- moved R4 147.9 mm to (87.5, 78.2), turned to 180 degrees
- moved C18 147.6 mm to (95.5, 57.5), turned to 180 degrees
- moved C35 146.7 mm to (95.3, 59.5), turned to 90 degrees
- moved C8 146.1 mm to (90.1, 67.7), turned to 90 degrees
- moved C47 142.0 mm to (91.4, 91.7), turned to 90 degrees
- moved C4 140.8 mm to (78.0, 59.5), turned to 90 degrees
- moved C7 140.3 mm to (92.3, 67.2), turned to 270 degrees
- moved C46 137.5 mm to (98.3, 77.5), turned to 90 degrees
- moved C43 134.8 mm to (95.3, 65.1), turned to 270 degrees
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Connections:
- C14 pad 2: Net-(C14-Pad2) -> +3V3
- C3 pad 2: +3.3VP -> +3V3
- C31 pad 2: Net-(C31-Pad2) -> +3V3
- C47 pad 1: Net-(C47-Pad1) -> NRST
- J3 pad 1: Net-(D11-Pad1) -> +3V3
- R11 pad 1: +3.3VP -> +3V3
- R18 pad 1: +3.3VP -> +3V3
- R24 pad 1: CHRG_READ -> Net-(R24-Pad1)
- R25 pad 2: +3V3 -> Net-(R25-Pad2)
- R27 pad 2: Net-(C10-Pad2) -> GND
- R33 pad 2: Net-(C47-Pad1) -> NRST
- R44 pad 2: PWR_LED -> PWR_LED_DIMM
- U1 pad 6: +3.3VP -> +3V3
- U11 pad 53: Net-(U11-Pad53) -> FLASH_WP
- U11 pad 7: Net-(C47-Pad1) -> NRST
- U2 pad 3: Net-(R3-Pad2) -> FLASH_WP
- U4 pad 1: Net-(R27-Pad1) -> Net-(R28-Pad2)
- U4 pad 2: VBUS -> Net-(R27-Pad1)
- U4 pad 3: Net-(Q7-Pad4) -> GND
- U4 pad 4: GND -> VBUS
- U4 pad 5: CHRG_READ -> Net-(C24-Pad1)
- U4 pad 6: Net-(C24-Pad1) -> Net-(R25-Pad2)
- U4 pad 8: Net-(R28-Pad2) -> Net-(R24-Pad1)
- U7 pad 4: Net-(C14-Pad2) -> +3V3
- U8 pad 1: Net-(C47-Pad1) -> NRST
- U9 pad 4: Net-(C31-Pad2) -> +3V3
Routing:
- net +3V3: track 0.00 -> 380.6 mm, vias 0 -> 28
- net SYSTEM_SCL: track 0.00 -> 118.4 mm, vias 0 -> 5
- net SYSTEM_SDA: track 0.00 -> 111.8 mm, vias 0 -> 7
- net VDD: track 0.00 -> 97.7 mm, vias 0 -> 6
- net GND: track 0.00 -> 83.4 mm, vias 0 -> 51
- net LED_TEMP: track 0.00 -> 69.7 mm, vias 0 -> 2
- net VBUS_ADC: track 0.00 -> 64.8 mm, vias 0 -> 6
- net BAT_TEMP: track 0.00 -> 60.0 mm, vias 0 -> 4
- net USB_DET: track 0.00 -> 59.4 mm, vias 0 -> 4
- net ETEMP_2: track 0.00 -> 59.0 mm, vias 0 -> 2
- net CHRH_PULL: track 0.00 -> 57.1 mm, vias 0 -> 1
- net CHRG_READ: track 0.00 -> 53.8 mm
- net Net-(J7-Pad6): track 0.00 -> 49.7 mm, vias 0 -> 1
- net PWR_KEEP: track 0.00 -> 49.4 mm, vias 0 -> 4
- net FLASH_WP: track 0.00 -> 47.6 mm, vias 0 -> 4
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- added copper zone on B.Cu, net GND
- added copper zone on F.Cu, net GND
Other:
- rule pad_to_mask_clearance: 0 -> 0.0508
- rule trace_min: 0.2 -> 0.2032
- rule via_min_size: 0.4 -> 0.3

Commit message: pcb update (not finished yet)
Parts:
- removed D12: LED_RGAB, Zasilacz_brama:LED_D5.0mm-4_RGB
- removed U6: ESP32-cam, Zasilacz_brama:ESP32-CAM
- added BZ1: Buzzer, Zasilacz_brama:PinHeader_1x02_P2.54mm_SMD, F.Cu at (32.7, 78.4)
- added C5: 22uF/10V, Capacitor_SMD:C_1210_3225Metric_Pad1.33x2.70mm_HandSolder, F.Cu at (58.9, 75.7)
- added D4: LED_RGCB, Zasilacz_brama:LED_D5.0mm-4_RGB, F.Cu at (97.7, 99.2)
- added Q7: BSS138, Package_TO_SOT_SMD:SOT-23, F.Cu at (42.0, 82.6)
- added R3: 1k, Resistor_SMD:R_0805_2012Metric_Pad1.20x1.40mm_HandSolder, F.Cu at (32.8, 84.7)
- added R34: 10k, Resistor_SMD:R_0805_2012Metric_Pad1.20x1.40mm_HandSolder, F.Cu at (37.4, 81.8)
- added R60: 0, Resistor_SMD:R_0805_2012Metric_Pad1.20x1.40mm_HandSolder, B.Cu at (66.2, 122.3)
- added Ue: ESP32-cam, Zasilacz_brama:ESP32-CAM, F.Cu at (86.5, 118.2)
- C14, C37, C39: moved to B.Cu
- moved C19 12.6 mm to (71.4, 98.1), turned to 180 degrees
- moved J4 9.09 mm to (76.8, 69.7)
- moved R9 6.10 mm to (60.5, 99.8), turned to 180 degrees
- moved R22 4.83 mm to (55.6, 107.9), turned to 0 degrees
- moved R56 4.64 mm to (92.5, 96.2), turned to 180 degrees
- moved C34 4.24 mm to (52.1, 121.1)
- moved R32 4.19 mm to (62.7, 73.2), turned to 90 degrees
- moved R43 3.53 mm to (64.8, 60.8), turned to 0 degrees
- moved R58 3.37 mm to (92.5, 100.1)
- moved R17 3.30 mm to (61.6, 102.9), turned to 90 degrees
- moved C39 3.24 mm to (72.4, 101.1)
- moved C25 3.22 mm to (91.2, 82.4)
- moved C36 2.71 mm to (60.3, 122.0)
- moved R50 2.71 mm to (58.3, 121.9)
- moved R49 2.69 mm to (56.3, 121.9)
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Connections:
- J7 pad 6: Net-(J7-Pad6) -> GND
- R32 pad 1: VDD -> VD
- U11 pad 54: Net-(U11-Pad54) -> BUZZER
- U7 pad 1: VDD -> VD
- XS1 pad 6: Net-(J7-Pad6) -> GND
Routing:
- net Net-(J7-Pad6): track 49.7 -> 0.00 mm, vias 1 -> 0
- net VDD: track 97.7 -> 132.4 mm
- net GND: track 83.4 -> 115.7 mm, vias 51 -> 78
- net +3V3: track 380.6 -> 357.6 mm, vias 28 -> 26
- net VBUS_ADC: track 64.8 -> 46.9 mm, vias 6 -> 4
- net Net-(J4-Pad1): track 13.6 -> 0.04 mm
- net BAT_TEMP: track 60.0 -> 71.2 mm
- net Net-(J1-Pad2): track 25.0 -> 18.3 mm
- net Net-(J7-Pad1): track 15.5 -> 22.1 mm
- net PWR_BUTTON: track 41.0 -> 46.4 mm
- net Net-(Q3-Pad3): track 24.5 -> 19.1 mm
- net BUZZER: track 0.00 -> 5.24 mm
- net Net-(J7-Pad2): track 15.1 -> 19.9 mm
- net USB_DET: track 59.4 -> 54.7 mm, vias 4 -> 2
- net Net-(C23-Pad1): track 15.6 -> 20.2 mm
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
Commit message: pcb final commit
Parts:
- removed BZ1: Buzzer, Zasilacz_brama:PinHeader_1x02_P2.54mm_SMD
- BT1, BT2: footprint Zasilacz_brama:BATT -> TinXsat:BATT
- D1, D2: moved to F.Cu
- D4: footprint Zasilacz_brama:LED_D5.0mm-4_RGB -> TinXsat:LED_D5.0mm-4_RGB
- J10, U12, U13, U14: footprint Zasilacz_brama:PinHeader_1x03_P2.00mm_SMD -> TinXsat:PinHeader_1x03_P2mm_SMD
- J2: footprint Zasilacz_brama:PinHeader_1x05_P2.54mm_SMD -> TinXsat:PinHeader_1x05_P2mm_SMD
- J3: footprint Zasilacz_brama:PinHeader_1x05_P2.54mm_SMD -> TinXsat:PinHeader_1x06_P2mm_SMD
- J5, J6, J9: footprint Zasilacz_brama:PinHeader_1x06_P2.00mm_SMD -> TinXsat:PinHeader_1x06_P2mm_SMD
- J7: footprint Zasilacz_brama:PinHeader_1x08_P2.00mm_SMD -> TinXsat:PinHeader_1x08_P2mm_SMD
- J8: footprint Zasilacz_brama:PinHeader_1x04_P2.54mm_SMD -> TinXsat:PinHeader_1x04_P2mm_SMD
- Q7, R3, R34: moved to B.Cu
- TH1: footprint Zasilacz_brama:PinHeader_1x02_P2.54mm_SMD -> TinXsat:PinHeader_1x02_P2mm_SMD
- U6: renamed from Ue; footprint Zasilacz_brama:ESP32-CAM -> TinXsat:ESP32-CAM
- moved R3 41.6 mm to (72.5, 72.5)
- moved Q7 33.1 mm to (72.5, 69.7), turned to 90 degrees
- moved R34 32.6 mm to (68.6, 72.5)
- moved R35 5.36 mm to (69.2, 73.0), turned to 90 degrees
- moved R4 3.15 mm to (90.2, 76.6), turned to 270 degrees
- moved D2 2.55 mm to (91.1, 75.6)
- moved D1 2.30 mm to (91.1, 73.6)
- moved C27 1.92 mm to (71.6, 68.5), turned to 270 degrees
- moved R2 1.92 mm to (86.1, 74.6)
- moved C18 0.78 mm to (96.2, 57.6)
- moved C22 0.78 mm to (96.2, 59.7)
- moved R13 0.77 mm to (82.8, 113.5)
- moved C41 0.37 mm to (79.7, 76.6)
- moved R12 0.22 mm to (82.8, 108.7)
- moved XS1 0.20 mm to (54.7, 86.6)
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Connections:
- Q7 pad 3: Net-(BZ1-Pad2) -> Net-(J3-Pad6)
- R1 pad 2: +3.3VP -> +3V3
Routing:
- net VDD: track 132.4 -> 68.4 mm, vias 6 -> 3
- net VD: track 0.00 -> 59.8 mm, vias 0 -> 4
- net GND: track 115.7 -> 150.4 mm, vias 78 -> 179
- net BUZZER: track 5.24 -> 32.2 mm, vias 0 -> 3
- net Net-(J3-Pad6): track 0.00 -> 21.3 mm, vias 0 -> 1
- net Net-(J4-Pad1): track 0.04 -> 14.9 mm
- net +3V3: track 357.6 -> 371.7 mm, vias 26 -> 32
- net PWR_LED_ON: track 44.1 -> 34.1 mm, vias 4 -> 2
- net Net-(D10-Pad1): track 30.1 -> 36.9 mm, vias 1 -> 2
- net DEBUG_LED_1: track 19.1 -> 25.4 mm
- net GPS_TX: track 41.6 -> 47.2 mm
- net Net-(Q7-Pad1): track 0.00 -> 5.34 mm
- net DEBUG_RX: track 38.1 -> 42.6 mm
- net USB_DET: track 54.7 -> 58.0 mm
- net Net-(R35-Pad2): track 6.89 -> 3.91 mm
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Other:
- outline, holes or cut-outs redrawn

Commit message: pcb gerber commit
Parts:
- added G***: LOGO, footprints:logo_pcbgogo, F.Cu at (75.5, 105.3)
- added G***: LOGO, footprints:logo, B.Cu at (58.5, 65.5)
- added REF**: OSHW-Logo_5.7x6mm_SilkScreen, Symbol:OSHW-Logo_5.7x6mm_SilkScreen, F.Cu at (75.4, 111.6)
- U2: footprint Package_SO:SOP-8_3.9x4.9mm_P1.27mm -> TinXsat:WSON-8-1EP_6x5mm_P1.27mm_EP3.4x4mm
- moved C7 8.27 mm to (88.0, 60.2), turned to 0 degrees
- moved R14 2.65 mm to (91.8, 60.2)
- moved C8 0.21 mm to (90.3, 67.8)
- moved R15 0.06 mm to (78.0, 55.6), turned to 90 degrees
Connections:
- R1 pad 2: +3V3 -> +3.3VP
- R15 pad 1: Net-(R15-Pad1) -> +3V3
- R15 pad 2: +3V3 -> Net-(R15-Pad2)
- U2 pad 7: Net-(U2-Pad7) -> Net-(R15-Pad2)
Routing:
- net GND: track 150.4 -> 158.6 mm, vias 179 -> 180
- net Net-(R15-Pad2): track 0.00 -> 2.65 mm
- net Net-(R14-Pad2): track 6.96 -> 9.29 mm
- net STM_USBDM: track 39.2 -> 38.4 mm
- net DEBUG_RX: track 42.6 -> 41.9 mm
- net DEBUG_TX: track 35.4 -> 34.8 mm
- net PWR_KEEP: track 51.6 -> 51.0 mm
- net PWR_BUTTON: track 46.4 -> 45.9 mm
- net VBUS_ADC: track 46.4 -> 45.9 mm
Other:
- board text added: "designed by Fifi 2020"

Commit message: pcb final commit after chinese changes
Parts:
- moved J9 0.37 mm to (98.0, 80.9)
- moved U13 0.30 mm to (69.4, 128.0)
- moved BT2 0.29 mm to (62.3, 127.5)
- moved BT1 0.27 mm to (88.1, 127.5)
- moved D4 0.23 mm to (97.5, 99.2)
- moved TH1 0.21 mm to (83.0, 128.0)
- moved J3 0.21 mm to (58.1, 52.0)
- moved J6 0.19 mm to (52.0, 64.0)
- moved U14 0.19 mm to (52.0, 61.5)
- moved U12 0.18 mm to (98.0, 61.5)
- moved J5 0.18 mm to (98.0, 64.0)
- moved J7 0.18 mm to (52.0, 78.8)
- moved J8 0.17 mm to (71.2, 52.0)
- moved J1 0.17 mm to (95.8, 107.5)
Connections:
- R1 pad 2: +3.3VP -> +3V3
Routing:
- net GND: track 158.6 -> 166.4 mm, vias 180 -> 178
- net BAT_TEMP: track 69.6 -> 66.5 mm
- net Net-(D10-Pad1): track 36.9 -> 34.1 mm
- net +3V3: track 372.1 -> 373.6 mm
- net Net-(J7-Pad1): track 22.1 -> 21.4 mm
Other:
- net class Default: clearance 0.2 -> 0.15
- rule trace_clearance: 0.2 -> 0.15
