File: electronics/TinXsat/TinXsat.sch (KiCad schematic (older format))
At the start: 54 parts

Commit message: pcb initial commit
Parts:
- removed C?: 22uF/10V, Capacitor_SMD:C_1210_3225Metric_Pad1.33x2.70mm_HandSolder, symbol Device:C
- removed D?: 1N4148W, Diode_SMD:D_SOD-123, symbol Diode:1N4148W
- added C1: 10n, Capacitor_SMD:C_0805_2012Metric_Pad1.18x1.45mm_HandSolder, symbol Device:C
- added C11: 2n2, Capacitor_SMD:C_0805_2012Metric_Pad1.18x1.45mm_HandSolder, symbol Device:C
- added C13, C15, C20, C45, C8: 22u, Capacitor_SMD:C_1210_3225Metric_Pad1.33x2.70mm_HandSolder, symbol Device:C
- added C14, C18, C19, C2, C22, C27, C3, C30, C33, C35, C37, C38, C39, C4, C40, C41, C42, C43, C46, C47, C7, C9: 100n, Capacitor_SMD:C_0805_2012Metric_Pad1.18x1.45mm_HandSolder, symbol Device:C
- added C21, C23, C32: 22uF/10V, Capacitor_SMD:C_1210_3225Metric_Pad1.33x2.70mm_HandSolder, symbol Device:C
- added C25, C28: 20p, Capacitor_SMD:C_0603_1608Metric_Pad1.08x0.95mm_HandSolder, symbol Device:C
- added C26, C29: 6p8, Capacitor_SMD:C_0603_1608Metric_Pad1.08x0.95mm_HandSolder, symbol Device:C
- added D1: GREEN, LED_SMD:LED_0805_2012Metric_Pad1.15x1.40mm_HandSolder, symbol Device:LED
- added D10, D3, D9: SMS240, Diode_SMD:D_MELF, symbol Diode:1N5711UR
- added D11: 1N4148, Diode_SMD:D_MiniMELF_Handsoldering, symbol Diode:1N4148
- added D12: LED_RGAB, Zasilacz_brama:LED_D5.0mm-4_RGB, symbol Device:LED_RGAB
- added D2: BLUE, LED_SMD:LED_0805_2012Metric_Pad1.15x1.40mm_HandSolder, symbol Device:LED
- added D4, D5: 4V7, Diode_SMD:D_MiniMELF_Handsoldering, symbol Device:D_Zener
- added D6: TXDIODE, LED_SMD:LED_0805_2012Metric_Pad1.15x1.40mm_HandSolder, symbol Device:LED
- added D7: RXDIODE, LED_SMD:LED_0805_2012Metric_Pad1.15x1.40mm_HandSolder, symbol Device:LED
- added F2, F3: Fuse, Fuse:Fuse_1206_3216Metric_Pad1.42x1.75mm_HandSolder, symbol Device:Fuse
- added J10: CAN, Connector_PinHeader_2.54mm:PinHeader_1x03_P2.54mm_Vertical, symbol Connector:Conn_01x03_Female
- added J2: ESP-PROG, Connector_PinHeader_2.54mm:PinHeader_1x05_P2.54mm_Vertical, symbol Connector:Conn_01x05_Female
- added J3: POWER_LED, Connector_PinHeader_2.54mm:PinHeader_1x05_P2.54mm_Vertical, symbol Connector:Conn_01x05_Female
- added J4: MCO_OUT, Connector_PinHeader_2.54mm:PinHeader_1x01_P2.54mm_Vertical, symbol Connector:Conn_01x01_Male
- added J5: BMP280_1, Connector_PinHeader_2.54mm:PinHeader_1x06_P2.54mm_Vertical, symbol Connector:Conn_01x06_Female
- added J6: BMP280_2, Connector_PinHeader_2.54mm:PinHeader_1x06_P2.54mm_Vertical, symbol Connector:Conn_01x06_Female
- added J7: Micro_SD_Card, Connector_Card:microSD_HC_Molex_104031-0811, symbol Connector:Micro_SD_Card
- added J8: GPS, Connector_PinHeader_2.54mm:PinHeader_1x04_P2.54mm_Vertical, symbol Connector:Conn_01x04_Female
- added J9: SWD, Connector_PinHeader_2.54mm:PinHeader_1x06_P2.54mm_Vertical, symbol Connector:Conn_01x06_Female
- added L2: 22uH/3A, Inductor_SMD:L_7.3x7.3_H3.5, symbol Device:L
- added L3: BEAD, Inductor_SMD:L_0805_2012Metric_Pad1.05x1.20mm_HandSolder, symbol Device:L
- added Q1: Si2371, Package_TO_SOT_SMD:SOT-23, symbol Transistor_FET:Si2371EDS
- added Q8: STD7NK40Z, Package_TO_SOT_SMD:TO-252-2, symbol Transistor_FET:STD7NK40Z
- added R1, R14, R15, R16, R3, R31, R33, R35, R45, R46, R47, R48: 10k, Resistor_SMD:R_0805_2012Metric_Pad1.20x1.40mm_HandSolder, symbol Device:R
- added R10, R8: 10, Resistor_SMD:R_0805_2012Metric_Pad1.20x1.40mm_HandSolder, symbol Device:R
- added R11, R18: 470, Resistor_SMD:R_0805_2012Metric_Pad1.20x1.40mm_HandSolder, symbol Device:R
- added R12, R13: N/M, Resistor_SMD:R_0805_2012Metric_Pad1.20x1.40mm_HandSolder, symbol Device:R
- added R2, R4, R56, R57, R58: 47, Resistor_SMD:R_0805_2012Metric_Pad1.20x1.40mm_HandSolder, symbol Device:R
- added R32: 22m, Resistor_SMD:R_MiniMELF_MMA-0204, symbol Device:R
- added R36, R39: 390, Resistor_SMD:R_0805_2012Metric_Pad1.20x1.40mm_HandSolder, symbol Device:R
- added R37, R40, R6, R7: 0, Resistor_SMD:R_0805_2012Metric_Pad1.20x1.40mm_HandSolder, symbol Device:R
- added R42, R43: R, Resistor_SMD:R_0805_2012Metric_Pad1.20x1.40mm_HandSolder, symbol Device:R
- added R44: 1k, Resistor_SMD:R_0805_2012Metric_Pad1.20x1.40mm_HandSolder, symbol Device:R
- added R52, R53: 2k2, Resistor_SMD:R_0805_2012Metric_Pad1.20x1.40mm_HandSolder, symbol Device:R
- added U1: CP2102N-A01-GQFN28, Package_DFN_QFN:QFN-28-1EP_5x5mm_P0.5mm_EP3.35x3.35mm, symbol Interface_USB:CP2102N-A01-GQFN28
- added U10: TPS61175PWP, Package_SO:HTSSOP-14-1EP_4.4x5mm_P0.65mm_EP3.4x5mm_Mask3x3.1mm_ThermalVias, symbol 2020-12-09_12-36-17:TPS61175PWP
- added U11: STM32F103RGTx, Package_QFP:LQFP-64_10x10mm_P0.5mm, symbol MCU_ST_STM32F1:STM32F103RGTx
- added U12, U13, U14: LM35-LP, Package_TO_SOT_THT:TO-92, symbol Sensor_Temperature:LM35-LP
- added U2: A25L032, Package_SO:SOP-8_3.9x4.9mm_P1.27mm, symbol sch-lib:A25L032
- added U3: MPU-6050, Sensor_Motion:InvenSense_QFN-24_4x4mm_P0.5mm, symbol Sensor_Motion:MPU-6050
- added U5: Ai-Thinker-Ra-01, RF_Module:Ai-Thinker-Ra-01-LoRa, symbol RF_Module:Ai-Thinker-Ra-01
- added U6: ESP32-cam, Zasilacz_brama:ESP32-CAM, symbol sch-lib:ESP32-cam
- added U7: INA219AxDCN, Package_TO_SOT_SMD:SOT-23-8, symbol Analog_ADC:INA219AxDCN
- added U8: MCP130, Package_TO_SOT_SMD:SOT-23, symbol Power_Supervisor:MCP130-xxxxTT
- added Y1: 8Mhz, Crystal:Crystal_HC49-U_Vertical, symbol Device:Crystal
- added Y2: 32768Hz, Crystal:Crystal_DS26_D2.0mm_L6.0mm_Horizontal_1EP_style1, symbol Device:Crystal
- BT1, BT2: renamed from BT?; footprint (none) -> Zasilacz_brama:BATT
- F1: renamed from F?; footprint (none) -> Fuse:Fuse_1206_3216Metric_Pad1.42x1.75mm_HandSolder
- J1: renamed from J?; footprint (none) -> Connector_USB:USB_Mini-B_Lumberg_2486_01_Horizontal
- R17, R19, R20, R21, R22, R23, R26, R29, R30, R5, R9: renamed from R?; footprint (none) -> Resistor_SMD:R_0805_2012Metric_Pad1.20x1.40mm_HandSolder
- R38: renamed from R?; footprint Resistor_SMD:R_MiniMELF_MMA-0204 -> Resistor_SMD:R_0805_2012Metric_Pad1.20x1.40mm_HandSolder
- SW1: renamed from SW?; footprint (none) -> Zasilacz_brama:Panasonic_EVQPUK_EVQPUB
- TH1: renamed from TH?; footprint (none) -> Connector_PinHeader_2.54mm:PinHeader_1x02_P2.54mm_Vertical
- gave numbers to parts that had none: 34
Connections:
- net labels added: +3.3VP, +VSW, BAT_TEMP, CAM-BSY, CAM-STROBE, DEBUG_LED_1, DEBUG_LED_2, DEBUG_RX, DEBUG_TX, ESP-RX, ESP-TX, ETEMP_1, ETEMP_2, FLASH_CS, GPS_RX, GPS_TX, GYRO_FRAME, GYRO_IRQ, GYRO_SCL, GYRO_SDA, LED_TEMP, LORA_CS, LORA_IRQ, LORA_RST, NRST, PWR_LED, PWR_LED_DIMM, PWR_LED_ON, SPI_MISO, SPI_MOSI, SPI_SCK, STATUS_LED_1, STATUS_LED_2, STATUS_LED_3, STM_USBDM, STM_USBDP, SWDCLK, SWDIO, SWO, SYSTEM_SCL, SYSTEM_SDA, UART_DM, UART_DP, USB_DET, VBUS_ADC
- wire segments 199 -> 679
- no-connect marks 0 -> 4
Other:
- note added: "3V3 SMPS"
- note added: "ADDR = 0x76\n"
- note added: "ADDR = 0x77\n\n"
- note added: "EDGE CONN"
- note added: "ESP-CAM\n"
- note added: "FLASH\n"
- note added: "GYRO"
- note added: "HSE"
- note added: "LORA"
- note added: "PWRLED DRIVER"
- note added: "PWRON LOGIC"
- note added: "SENSORS"
- note added: "STM32"
- note added: "USB & CHARGING"
- note added: "USB/UART BRIDGE"
- note added: "USB_DM = CANRX\nUSB_DP = CANTX"
- note removed: "This diode is here to ensure only current \nsink from pin (pull up) no current source, \nso MCU won't power up from this voltage"
- moved on the sheet: BT1, BT2, C10, C12, C16, C17, C24, C31, C34, C36, C44, C6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

Commit message: pcb initial commit
Parts:
- removed C10: 470n, Capacitor_SMD:C_0805_2012Metric_Pad1.18x1.45mm_HandSolder, symbol Device:C
- removed C21: 22uF/10V, Capacitor_SMD:C_1210_3225Metric_Pad1.33x2.70mm_HandSolder, symbol Device:C
- removed D11: 1N4148, Diode_SMD:D_MiniMELF_Handsoldering, symbol Diode:1N4148
- removed D4, D5: 4V7, Diode_SMD:D_MiniMELF_Handsoldering, symbol Device:D_Zener
- removed D8: SMS240, Diode_SMD:D_MELF, symbol Diode:1N5711UR
- removed J7: Micro_SD_Card, Connector_Card:microSD_HC_Molex_104031-0811, symbol Connector:Micro_SD_Card
- removed L1: 4.7uH/2.9A, Inductor_SMD:L_7.3x7.3_H3.5, symbol Device:L
- removed Q7: IRF7406, Package_SO:SOIC-8_3.9x4.9mm_P1.27mm, symbol Transistor_FET:IRF7404
- removed R3: 10k, Resistor_SMD:R_0805_2012Metric_Pad1.20x1.40mm_HandSolder, symbol Device:R
- removed R34: 100m, Resistor_SMD:R_MiniMELF_MMA-0204, symbol Device:R
- removed U4: LTC4002ES8-4.2, Package_SO:SOIC-8_3.9x4.9mm_P1.27mm, symbol Battery_Management:LTC4002ES8-4.2
- added J7: ESP-card, Zasilacz_brama:PinHeader_1x08_P2.00mm_SMD, symbol Connector:Conn_01x09_Female
- added U4: TP4056, Package_SO:SOIC-8-1EP_3.9x4.9mm_P1.27mm_EP2.29x3mm, symbol tp4056:TP4056
- added XS1: SD_ebay-uSD-push_push_SMD, footprints:Conn_uSDcard, symbol uSD_push-push_ebay:SD_ebay-uSD-push_push_SMD
- C17, C24, C34: value 22uF/10V -> 10uF/10V; footprint Capacitor_SMD:C_1210_3225Metric_Pad1.33x2.70mm_HandSolder -> Capacitor_SMD:C_1206_3216Metric_Pad1.33x1.80mm_HandSolder
- C45, C8: value 22u -> 10u; footprint Capacitor_SMD:C_1210_3225Metric_Pad1.33x2.70mm_HandSolder -> Capacitor_SMD:C_1206_3216Metric_Pad1.33x1.80mm_HandSolder
- J10: footprint Connector_PinHeader_2.54mm:PinHeader_1x03_P2.54mm_Vertical -> Zasilacz_brama:PinHeader_1x03_P2.00mm_SMD
- J2, J3: footprint Connector_PinHeader_2.54mm:PinHeader_1x05_P2.54mm_Vertical -> Zasilacz_brama:PinHeader_1x05_P2.54mm_SMD
- J5, J6, J9: footprint Connector_PinHeader_2.54mm:PinHeader_1x06_P2.54mm_Vertical -> Zasilacz_brama:PinHeader_1x06_P2.00mm_SMD
- J8: footprint Connector_PinHeader_2.54mm:PinHeader_1x04_P2.54mm_Vertical -> Zasilacz_brama:PinHeader_1x04_P2.54mm_SMD
- R25: value 390k -> 10k
- R59: footprint Resistor_SMD:R_MiniMELF_MMA-0204 -> Resistor_SMD:R_0805_2012Metric_Pad1.20x1.40mm_HandSolder
- SW1: footprint Zasilacz_brama:Panasonic_EVQPUK_EVQPUB -> Button_Switch_THT:SW_Tactile_SKHH_Angled
- TH1: footprint Connector_PinHeader_2.54mm:PinHeader_1x02_P2.54mm_Vertical -> Zasilacz_brama:PinHeader_1x02_P2.54mm_SMD
- U10: footprint Package_SO:HTSSOP-14-1EP_4.4x5mm_P0.65mm_EP3.4x5mm_Mask3x3.1mm_ThermalVias -> footprints:TPS61175PWP
- U12, U13, U14: footprint Package_TO_SOT_THT:TO-92 -> Zasilacz_brama:PinHeader_1x03_P2.00mm_SMD
- Y1: footprint Crystal:Crystal_HC49-U_Vertical -> Crystal:Crystal_SMD_HC49-SD
Connections:
- net labels added: FLASH_WP
- net labels removed: PWR_LED
- wire segments 679 -> 678
Other:
- note removed: "Rsh=100mV/1A=0,01Ohm"
- moved on the sheet: C16, C17, R24, R28, TH1

Commit message: pcb update (not finished yet)
Parts:
- removed D12: LED_RGAB, Zasilacz_brama:LED_D5.0mm-4_RGB, symbol Device:LED_RGAB
- added BZ1: Buzzer, Zasilacz_brama:PinHeader_1x02_P2.54mm_SMD, symbol Device:Buzzer
- added C5: 22uF/10V, Capacitor_SMD:C_1210_3225Metric_Pad1.33x2.70mm_HandSolder, symbol Device:C
- added D4: LED_RGCB, Zasilacz_brama:LED_D5.0mm-4_RGB, symbol Device:LED_RGCB
- added Q7: BSS138, Package_TO_SOT_SMD:SOT-23, symbol Transistor_FET:BSS138
- added R3: 1k, Resistor_SMD:R_0805_2012Metric_Pad1.20x1.40mm_HandSolder, symbol Device:R
- added R34: 10k, Resistor_SMD:R_0805_2012Metric_Pad1.20x1.40mm_HandSolder, symbol Device:R
- added R60: 0, Resistor_SMD:R_0805_2012Metric_Pad1.20x1.40mm_HandSolder, symbol Device:R
Connections:
- net labels added: BUZZER, VD
- wire segments 678 -> 697
- no-connect marks 4 -> 3
Changed lines of the file:
@@
 $EndComp
 $Comp
-L power:VDD #PWR0128
-U 1 1 60024C84
-P 13600 1750
-F 0 "#PWR0128" H 13600 1600 50  0001 C CNN
-F 1 "VDD" H 13615 1923 50  0000 C CNN
-F 2 "" H 13600 1750 50  0001 C CNN
-F 3 "" H 13600 1750 50  0001 C CNN
-	1    13600 1750
-	1    0    0    -1
-$EndComp
-$Comp
 L power:+3V3 #PWR0129
 U 1 1 600256E8
@@
 Connection ~ 9500 2500
 Wire Wire Line
-	9500 2500 10500 2500
+	9500 2500 9750 2500
 $Comp
 L Device:Fuse F2
@@
 	21200 8900 21200 8950
 NoConn ~ 12050 8350
-NoConn ~ 12050 7750
 Text GLabel 12000 7950 0    50   Input ~ 0
 LED_TEMP
@@
 Wire Wire Line
 	10650 14750 10650 14800
-$Comp
-L power:VDD #PWR0207
-U 1 1 62469EA7
-P 10350 13450
-F 0 "#PWR0207" H 10350 13300 50  0001 C CNN
-F 1 "VDD" H 10365 13623 50  0000 C CNN
-F 2 "" H 10350 13450 50  0001 C CNN
-F 3 "" H 10350 13450 50  0001 C CNN
-	1    10350 13450
-	1    0    0    -1
-$EndComp
 Wire Wire Line
 	10350 13450 10350 13650
@@
 U 1 1 625B821A
 P 11750 13850
-F 0 "C23" H 11865 13896 50  0000 L CNN
-F 1 "22uF/10V" H 11865 13805 50  0000 L CNN
+F 0 "C23" H 11800 13950 50  0000 L CNN
+F 1 "22uF/10V" H 11800 13750 50  0000 L CNN
 F 2 "Capacitor_SMD:C_1210_3225Metric_Pad1.33x2.70mm_HandSolder" H 11788 13700 50  0001 C CNN
 F 3 "~" H 11750 13850 50  0001 C CNN
@@
 	14050 7050 13450 7050
 Wire Wire Line
-	21900 10350 21900 10250
-Wire Wire Line
 	21800 10350 21900 10350
-$Comp
-L Device:LED_RGAB D12
-U 1 1 60BE6889
-P 21600 10350
-F 0 "D12" H 21600 10847 50  0000 C CNN
-F 1 "LED_RGAB" H 21600 10756 50  0000 C CNN
-F 2 "Zasilacz_brama:LED_D5.0mm-4_RGB" H 21600 10300 50  0001 C CNN
-F 3 "~" H 21600 10300 50  0001 C CNN
-	1    21600 10350
-	1    0    0    -1
-$EndComp
 Text GLabel 17600 8750 2    50   Input ~ 0
 ETEMP_1
@@
 Text GLabel 20900 10150 0    50   Input ~ 0
 STATUS_LED_1
-$Comp
-L power:+3V3 #PWR0154
-U 1 1 5FD28F05
-P 21900 10250
-F 0 "#PWR0154" H 21900 10100 50  0001 C CNN
-F 1 "+3V3" H 21915 10423 50  0000 C CNN
-F 2 "" H 21900 10250 50  0001 C CNN
-F 3 "" H 21900 10250 50  0001 C CNN
-	1    21900 10250
-	1    0    0    -1
-$EndComp
 Text GLabel 17600 6200 2    50   Input ~ 0
 BAT_TEMP
@@
 Wire Wire Line
 	11750 14000 11750 14100
-Wire Wire Line
-	10950 13650 11750 13650
 $Comp
 L Connector:Conn_01x09_Female J7
@@
 	1    0    0    -1
 $EndComp
+Text GLabel 12000 7750 0    50   Input ~ 0
+BUZZER
+Wire Wire Line
+	12000 7750 12050 7750
+Text GLabel 20500 14000 0    50   Input ~ 0
+BUZZER
+$Comp
+L Device:Buzzer BZ1
+U 1 1 5FF0BA17
+P 21450 13650
+F 0 "BZ1" H 21602 13679 50  0000 L CNN
+F 1 "Buzzer" H 21602 13588 50  0000 L CNN
+F 2 "Zasilacz_brama:PinHeader_1x02_P2.54mm_SMD" V 21425 13750 50  0001 C CNN
+F 3 "~" V 21425 13750 50  0001 C CNN
+	1    21450 13650
+	1    0    0    -1
+$EndComp
+$Comp
+L Transistor_FET:BSS138 Q7
+U 1 1 5FF0D389
+P 21200 14000
+F 0 "Q7" H 21404 14046 50  0000 L CNN
+F 1 "BSS138" H 21404 13955 50  0000 L CNN
+F 2 "Package_TO_SOT_SMD:SOT-23" H 21400 13925 50  0001 L CIN
+F 3 "https://www.onsemi.com/pub/Collateral/BSS138-D.PDF" H 21200 14000 50  0001 L CNN
+	1    21200 14000
+	1    0    0    -1
+$EndComp
+$Comp
+L Device:R R3
+U 1 1 5FF100CC
+P 20750 14000
+F 0 "R3" V 20543 14000 50  0000 C CNN
+F 1 "1k" V 20634 14000 50  0000 C CNN
+F 2 "Resistor_SMD:R_0805_2012Metric_Pad1.20x1.40mm_HandSolder" V 20680 14000 50  0001 C CNN
+F 3 "~" H 20750 14000 50  0001 C CNN
+	1    20750 14000
+	0    1    1    0
+$EndComp
+$Comp
+L Device:R R34
+U 1 1 5FF11CEF
+P 20950 14200
+F 0 "R34" H 20880 14154 50  0000 R CNN
+F 1 "10k" H 20880 14245 50  0000 R CNN
+F 2 "Resistor_SMD:R_0805_2012Metric_Pad1.20x1.40mm_HandSolder" V 20880 14200 50  0001 C CNN
+F 3 "~" H 20950 14200 50  0001 C CNN
+	1    20950 14200
+	-1   0    0    1
+$EndComp
+Wire Wire Line
+	20900 14000 20950 14000
+Wire Wire Line
+	20950 14000 20950 14050
+Connection ~ 20950 14000
+Wire Wire Line
+	20950 14000 21000 14000
+Wire Wire Line
+	20950 14350 20950 14400
+Wire Wire Line
+	20950 14400 21300 14400
+Wire Wire Line
+	21300 14400 21300 14200
+$Comp
+L power:GND #PWR0158
+U 1 1 600B6588
+P 21300 14450
+F 0 "#PWR0158" H 21300 14200 50  0001 C CNN
+F 1 "GND" H 21305 14277 50  0000 C CNN
+F 2 "" H 21300 14450 50  0001 C CNN
+F 3 "" H 21300 14450 50  0001 C CNN
+	1    21300 14450
+	1    0    0    -1
+$EndComp
+Wire Wire Line
+	21300 14450 21300 14400
+Connection ~ 21300 14400
+Wire Wire Line
+	20600 14000 20500 14000
+$Comp
+L power:+VSW #PWR0200
+U 1 1 601D1A50
+P 21300 13500
+F 0 "#PWR0200" H 21300 13350 50  0001 C CNN
+F 1 "+VSW" H 21315 13673 50  0000 C CNN
+F 2 "" H 21300 13500 50  0001 C CNN
+F 3 "" H 21300 13500 50  0001 C CNN
+	1    21300 13500
+	1    0    0    -1
+$EndComp
+Wire Wire Line
+	21300 13500 21300 13550
+Wire Wire Line
+	21300 13550 21350 13550
+Wire Wire Line
+	21300 13750 21350 13750
+Wire Wire Line
+	21300 13750 21300 13800
+$Comp
+L power:VD #PWR0203
+U 1 1 6041EEBA
+P 9750 2100
+F 0 "#PWR0203" H 9750 1950 50  0001 C CNN
+F 1 "VD" H 9765 2273 50  0000 C CNN
+F 2 "" H 9750 2100 50  0001 C CNN
+F 3 "" H 9750 2100 50  0001 C CNN
+	1    9750 2100
+	1    0    0    -1
+$EndComp
+$Comp
+L Device:R R60
+U 1 1 60426032
+P 9750 2300
+F 0 "R60" H 9680 2254 50  0000 R CNN
+F 1 "0" H 9680 2345 50  0000 R CNN
+F 2 "Resistor_SMD:R_0805_2012Metric_Pad1.20x1.40mm_HandSolder" V 9680 2300 50  0001 C CNN
+F 3 "~" H 9750 2300 50  0001 C CNN
+	1    9750 2300
+	-1   0    0    1
+$EndComp
+Wire Wire Line
+	9750 2100 9750 2150
+Wire Wire Line
+	9750 2450 9750 2500
+Connection ~ 9750 2500
+Wire Wire Line
+	9750 2500 10500 2500
+$Comp
+L power:VD #PWR0207
+U 1 1 6054222C
+P 10350 13450
+F 0 "#PWR0207" H 10350 13300 50  0001 C CNN
+F 1 "VD" H 10365 13623 50  0000 C CNN
+F 2 "" H 10350 13450 50  0001 C CNN
+F 3 "" H 10350 13450 50  0001 C CNN
+	1    10350 13450
+	1    0    0    -1
+$EndComp
+$Comp
+L Device:C C5
+U 1 1 6054B671
+P 11450 13850
+F 0 "C5" H 11250 13950 50  0000 L CNN
+F 1 "22uF/10V" H 11050 13750 50  0000 L CNN
+F 2 "Capacitor_SMD:C_1210_3225Metric_Pad1.33x2.70mm_HandSolder" H 11488 13700 50  0001 C CNN
+F 3 "~" H 11450 13850 50  0001 C CNN
+	1    11450 13850
+	1    0    0    -1
+$EndComp
+$Comp
+L power:GND #PWR0218
+U 1 1 6054B677
+P 11450 14100
+F 0 "#PWR0218" H 11450 13850 50  0001 C CNN
+F 1 "GND" H 11455 13927 50  0000 C CNN
+F 2 "" H 11450 14100 50  0001 C CNN
+F 3 "" H 11450 14100 50  0001 C CNN
+	1    11450 14100
+	-1   0    0    -1
+$EndComp
+Wire Wire Line
+	11450 13700 11450 13650
+Wire Wire Line
+	11450 14000 11450 14100
+Wire Wire Line
+	10950 13650 11450 13650
+Connection ~ 11450 13650
+Wire Wire Line
+	11450 13650 11750 13650
+$Comp
+L power:GND #PWR0219
+U 1 1 5FF2DAEA
+P 5100 4500
+F 0 "#PWR0219" H 5100 4250 50  0001 C CNN
+F 1 "GND" H 5105 4327 50  0000 C CNN
+F 2 "" H 5100 4500 50  0001 C CNN
+F 3 "" H 5100 4500 50  0001 C CNN
+	1    5100 4500
+	1    0    0    -1
+$EndComp
+Connection ~ 5100 4500
+$Comp
+L power:VDD #PWR0128
+U 1 1 60024C84
+P 13600 1750
+F 0 "#PWR0128" H 13600 1600 50  0001 C CNN
+F 1 "VDD" H 13615 1923 50  0000 C CNN
+F 2 "" H 13600 1750 50  0001 C CNN
+F 3 "" H 13600 1750 50  0001 C CNN
+	1    13600 1750
+	1    0    0    -1
+$EndComp
+$Comp
+L Device:LED_RGCB D4
+U 1 1 60074E3E
+P 21600 10350
+F 0 "D4" H 21600 9883 50  0000 C CNN
+F 1 "LED_RGCB" H 21600 9974 50  0000 C CNN
+F 2 "Zasilacz_brama:LED_D5.0mm-4_RGB" H 21600 10300 50  0001 C CNN
+F 3 "~" H 21600 10300 50  0001 C CNN
+	1    21600 10350
+	-1   0    0    1
+$EndComp
+$Comp
+L power:GND #PWR0154
+U 1 1 60078C02
+P 21900 10400
+F 0 "#PWR0154" H 21900 10150 50  0001 C CNN
+F 1 "GND" H 21905 10227 50  0000 C CNN
+F 2 "" H 21900 10400 50  0001 C CNN
+F 3 "" H 21900 10400 50  0001 C CNN
+	1    21900 10400
+	1    0    0    -1
+$EndComp
+Wire Wire Line
+	21900 10350 21900 10400
 $EndSCHEMATC
