File: electronics/TinXsat/TinXsat.sch (KiCad schematic (older format))
At the start: 160 parts, among them J1 USB_B_Mini, J10 CAN, J2 ESP-PROG, J3 POWER_LED, J4 MCO_OUT, J5 BMP280_1, J6 BMP280_2, J7 ESP-card, J8 GPS, J9 SWD, Q1 Si2371, Q2 Si2371, Q3 BSS138, Q4 BSS138, Q5 Si2371, Q6 BSS138, Q7 BSS138, Q8 STD7NK40Z, SW1 SW_Push, U1 CP2102N-A01-GQFN28, U10 TPS61175PWP, U11 STM32F103RGTx, U12 LM35-LP, U13 LM35-LP, U14 LM35-LP, U15 TPS63001, U2 A25L032, U3 MPU-6050, U4 TP4056, U5 Ai-Thinker-Ra-01, U6 ESP32-cam, U7 INA219AxDCN, U8 MCP130, U9 INA219AxDCN, Y1 8Mhz, Y2 32768Hz

Commit message: pcb final commit
Parts:
- removed BZ1: Buzzer, Zasilacz_brama:PinHeader_1x02_P2.54mm_SMD, symbol Device:Buzzer
- removed J3: POWER_LED, Zasilacz_brama:PinHeader_1x05_P2.54mm_SMD, symbol Connector:Conn_01x05_Female
- added J3: POWER_LED, TinXsat:PinHeader_1x06_P2mm_SMD, symbol Connector:Conn_01x06_Female
- BT1, BT2: footprint Zasilacz_brama:BATT -> TinXsat:BATT
- D4: footprint Zasilacz_brama:LED_D5.0mm-4_RGB -> TinXsat:LED_D5.0mm-4_RGB
- J10, U12, U13, U14: footprint Zasilacz_brama:PinHeader_1x03_P2.00mm_SMD -> TinXsat:PinHeader_1x03_P2mm_SMD
- J2: footprint Zasilacz_brama:PinHeader_1x05_P2.54mm_SMD -> TinXsat:PinHeader_1x05_P2mm_SMD
- J5, J6, J9: footprint Zasilacz_brama:PinHeader_1x06_P2.00mm_SMD -> TinXsat:PinHeader_1x06_P2mm_SMD
- J7: footprint Zasilacz_brama:PinHeader_1x08_P2.00mm_SMD -> TinXsat:PinHeader_1x08_P2mm_SMD
- J8: footprint Zasilacz_brama:PinHeader_1x04_P2.54mm_SMD -> TinXsat:PinHeader_1x04_P2mm_SMD
- TH1: footprint Zasilacz_brama:PinHeader_1x02_P2.54mm_SMD -> TinXsat:PinHeader_1x02_P2mm_SMD
- U6: footprint Zasilacz_brama:ESP32-CAM -> TinXsat:ESP32-CAM
Connections:
- net +3V3: now also J3.1 (Pin_1)
- net +VSW: now also J3.4 (Pin_4)
- net GND: now also J3.3 (Pin_3)
- net LED_TEMP: now also J3.2 (Pin_2)
- net at Q7.3 (D): now also J3.6 (Pin_6)
- net at Q8.2 (D): now also J3.5 (Pin_5)
- no-connect marks 3 -> 8
Changed lines of the file:
@@
 F 0 "BT2" H 11018 3196 50  0000 L CNN
 F 1 "LiOn" H 11018 3105 50  0000 L CNN
-F 2 "Zasilacz_brama:BATT" V 10900 3160 50  0001 C CNN
+F 2 "TinXsat:BATT" V 10900 3160 50  0001 C CNN
 F 3 "~" V 10900 3160 50  0001 C CNN
 	1    10900 3100
@@
 F 0 "BT1" H 10618 3196 50  0000 L CNN
 F 1 "LiOn" H 10618 3105 50  0000 L CNN
-F 2 "Zasilacz_brama:BATT" V 10500 3160 50  0001 C CNN
+F 2 "TinXsat:BATT" V 10500 3160 50  0001 C CNN
 F 3 "~" V 10500 3160 50  0001 C CNN
 	1    10500 3100
@@
 F 0 "TH1" H 8147 3446 50  0000 L CNN
 F 1 "BAT_NTC" H 8147 3355 50  0000 L CNN
-F 2 "Zasilacz_brama:PinHeader_1x02_P2.54mm_SMD" H 8050 3450 50  0001 C CNN
+F 2 "TinXsat:PinHeader_1x02_P2mm_SMD" H 8050 3450 50  0001 C CNN
 F 3 "~" H 8050 3450 50  0001 C CNN
 	1    8050 3400
@@
 F 0 "J9" H 21428 6176 50  0000 L CNN
 F 1 "SWD" H 21428 6085 50  0000 L CNN
-F 2 "Zasilacz_brama:PinHeader_1x06_P2.00mm_SMD" H 21400 6200 50  0001 C CNN
+F 2 "TinXsat:PinHeader_1x06_P2mm_SMD" H 21400 6200 50  0001 C CNN
 F 3 "~" H 21400 6200 50  0001 C CNN
 	1    21400 6200
@@
 F 0 "J10" H 21428 7626 50  0000 L CNN
 F 1 "CAN" H 21428 7535 50  0000 L CNN
-F 2 "Zasilacz_brama:PinHeader_1x03_P2.00mm_SMD" H 21400 7600 50  0001 C CNN
+F 2 "TinXsat:PinHeader_1x03_P2mm_SMD" H 21400 7600 50  0001 C CNN
 F 3 "~" H 21400 7600 50  0001 C CNN
 	1    21400 7600
@@
 F 0 "J5" H 18478 9826 50  0000 L CNN
 F 1 "BMP280_1" H 18478 9735 50  0000 L CNN
-F 2 "Zasilacz_brama:PinHeader_1x06_P2.00mm_SMD" H 18450 9850 50  0001 C CNN
+F 2 "TinXsat:PinHeader_1x06_P2mm_SMD" H 18450 9850 50  0001 C CNN
 F 3 "~" H 18450 9850 50  0001 C CNN
 	1    18450 9850
@@
 F 0 "J6" H 18478 10476 50  0000 L CNN
 F 1 "BMP280_2" H 18478 10385 50  0000 L CNN
-F 2 "Zasilacz_brama:PinHeader_1x06_P2.00mm_SMD" H 18450 10500 50  0001 C CNN
+F 2 "TinXsat:PinHeader_1x06_P2mm_SMD" H 18450 10500 50  0001 C CNN
 F 3 "~" H 18450 10500 50  0001 C CNN
 	1    18450 10500
@@
 F 0 "U6" H 6700 7150 50  0000 C CNN
 F 1 "ESP32-cam" H 6750 7050 50  0000 C CNN
-F 2 "Zasilacz_brama:ESP32-CAM" H 6450 6550 50  0001 C CNN
+F 2 "TinXsat:ESP32-CAM" H 6450 6550 50  0001 C CNN
 F 3 "" H 6450 6550 50  0001 C CNN
 	1    6450 6550
@@
 F 0 "J8" H 21478 8676 50  0000 L CNN
 F 1 "GPS" H 21478 8585 50  0000 L CNN
-F 2 "Zasilacz_brama:PinHeader_1x04_P2.54mm_SMD" H 21450 8700 50  0001 C CNN
+F 2 "TinXsat:PinHeader_1x04_P2mm_SMD" H 21450 8700 50  0001 C CNN
 F 3 "~" H 21450 8700 50  0001 C CNN
 	1    21450 8700
@@
 F 0 "U12" H 16821 8796 50  0000 R CNN
 F 1 "LM35-LP" H 16821 8705 50  0000 R CNN
-F 2 "Zasilacz_brama:PinHeader_1x03_P2.00mm_SMD" H 17200 8500 50  0001 L CNN
+F 2 "TinXsat:PinHeader_1x03_P2mm_SMD" H 17200 8500 50  0001 L CNN
 F 3 "http://www.ti.com/lit/ds/symlink/lm35.pdf" H 17150 8750 50  0001 C CNN
 	1    17150 8750
@@
 F 0 "U14" H 16821 7496 50  0000 R CNN
 F 1 "LM35-LP" H 16821 7405 50  0000 R CNN
-F 2 "Zasilacz_brama:PinHeader_1x03_P2.00mm_SMD" H 17200 7200 50  0001 L CNN
+F 2 "TinXsat:PinHeader_1x03_P2mm_SMD" H 17200 7200 50  0001 L CNN
 F 3 "http://www.ti.com/lit/ds/symlink/lm35.pdf" H 17150 7450 50  0001 C CNN
 	1    17150 7450
@@
 LED_TEMP
 $Comp
-L Connector:Conn_01x05_Female J3
-U 1 1 6140FF74
-P 21750 12100
-F 0 "J3" H 21778 12126 50  0000 L CNN
-F 1 "POWER_LED" H 21778 12035 50  0000 L CNN
-F 2 "Zasilacz_brama:PinHeader_1x05_P2.54mm_SMD" H 21750 12100 50  0001 C CNN
-F 3 "~" H 21750 12100 50  0001 C CNN
-	1    21750 12100
-	1    0    0    -1
-$EndComp
-$Comp
 L power:+3V3 #PWR0191
 U 1 1 6142098D
@@
 F 0 "U13" H 16821 6246 50  0000 R CNN
 F 1 "LM35-LP" H 16821 6155 50  0000 R CNN
-F 2 "Zasilacz_brama:PinHeader_1x03_P2.00mm_SMD" H 17200 5950 50  0001 L CNN
+F 2 "TinXsat:PinHeader_1x03_P2mm_SMD" H 17200 5950 50  0001 L CNN
 F 3 "http://www.ti.com/lit/ds/symlink/lm35.pdf" H 17150 6200 50  0001 C CNN
 	1    17150 6200
@@
 F 0 "J2" H 8228 6626 50  0000 L CNN
 F 1 "ESP-PROG" H 8228 6535 50  0000 L CNN
-F 2 "Zasilacz_brama:PinHeader_1x05_P2.54mm_SMD" H 8200 6600 50  0001 C CNN
+F 2 "TinXsat:PinHeader_1x05_P2mm_SMD" H 8200 6600 50  0001 C CNN
 F 3 "~" H 8200 6600 50  0001 C CNN
 	1    8200 6600
@@
 F 0 "J7" H 5728 3876 50  0000 L CNN
 F 1 "ESP-card" H 5728 3785 50  0000 L CNN
-F 2 "Zasilacz_brama:PinHeader_1x08_P2.00mm_SMD" H 5700 3850 50  0001 C CNN
+F 2 "TinXsat:PinHeader_1x08_P2mm_SMD" H 5700 3850 50  0001 C CNN
 F 3 "~" H 5700 3850 50  0001 C CNN
 	1    5700 3850
@@
 BUZZER
 $Comp
-L Device:Buzzer BZ1
-U 1 1 5FF0BA17
-P 21450 13650
-F 0 "BZ1" H 21602 13679 50  0000 L CNN
-F 1 "Buzzer" H 21602 13588 50  0000 L CNN
-F 2 "Zasilacz_brama:PinHeader_1x02_P2.54mm_SMD" V 21425 13750 50  0001 C CNN
-F 3 "~" V 21425 13750 50  0001 C CNN
-	1    21450 13650
-	1    0    0    -1
-$EndComp
-$Comp
 L Transistor_FET:BSS138 Q7
 U 1 1 5FF0D389
@@
 	20600 14000 20500 14000
 $Comp
-L power:+VSW #PWR0200
-U 1 1 601D1A50
-P 21300 13500
-F 0 "#PWR0200" H 21300 13350 50  0001 C CNN
-F 1 "+VSW" H 21315 13673 50  0000 C CNN
-F 2 "" H 21300 13500 50  0001 C CNN
-F 3 "" H 21300 13500 50  0001 C CNN
-	1    21300 13500
-	1    0    0    -1
-$EndComp
-Wire Wire Line
-	21300 13500 21300 13550
-Wire Wire Line
-	21300 13550 21350 13550
-Wire Wire Line
-	21300 13750 21350 13750
-Wire Wire Line
-	21300 13750 21300 13800
-$Comp
 L power:VD #PWR0203
 U 1 1 6041EEBA
@@
 F 0 "D4" H 21600 9883 50  0000 C CNN
 F 1 "LED_RGCB" H 21600 9974 50  0000 C CNN
-F 2 "Zasilacz_brama:LED_D5.0mm-4_RGB" H 21600 10300 50  0001 C CNN
+F 2 "TinXsat:LED_D5.0mm-4_RGB" H 21600 10300 50  0001 C CNN
 F 3 "~" H 21600 10300 50  0001 C CNN
 	1    21600 10350
@@
 Wire Wire Line
 	21900 10350 21900 10400
+NoConn ~ 7400 6600
+NoConn ~ 6450 6200
+NoConn ~ 6450 6700
+NoConn ~ 6450 6800
+NoConn ~ 6450 6900
+$Comp
+L Connector:Conn_01x06_Female J3
+U 1 1 5FE90EA7
+P 21750 12100
+F 0 "J3" H 21778 12076 50  0000 L CNN
+F 1 "POWER_LED" H 21778 11985 50  0000 L CNN
+F 2 "TinXsat:PinHeader_1x06_P2mm_SMD" H 21750 12100 50  0001 C CNN
+F 3 "~" H 21750 12100 50  0001 C CNN
+	1    21750 12100
+	1    0    0    -1
+$EndComp
+Wire Wire Line
+	21550 12400 21450 12400
+Wire Wire Line
+	21450 12400 21450 13600
+Wire Wire Line
+	21450 13600 21300 13600
+Wire Wire Line
+	21300 13600 21300 13800
 $EndSCHEMATC

Commit message: pcb gerber commit
Parts:
- U2: footprint Package_SO:SOP-8_3.9x4.9mm_P1.27mm -> TinXsat:WSON-8-1EP_6x5mm_P1.27mm_EP3.4x4mm
Connections:
- net +3V3: now also R15.1; no longer R15.2
- net at U2.7 (HOLD): now also R15.2; no longer R15.1
Changed lines of the file:
@@
 FLASH_WP
-$Comp
-L sch-lib:A25L032 U2
-U 1 1 60070B82
-P 2250 6750
-F 0 "U2" H 1900 7250 50  0000 C CNN
-F 1 "A25L032" H 2000 7150 50  0000 C CNN
-F 2 "Package_SO:SOP-8_3.9x4.9mm_P1.27mm" H 2250 6150 50  0001 C CNN
-F 3 "http://www.elm-tech.com/en/products/spi-flash-memory/gd25d10/gd25d10.pdf" H 2250 6750 50  0001 C CNN
-	1    2250 6750
-	1    0    0    -1
-$EndComp
 $Comp
 L power:GND #PWR0162
@@
 	1700 6750 1750 6750
 $Comp
-L Device:R R15
-U 1 1 60255FDC
-P 3000 6800
-F 0 "R15" V 2900 6800 50  0000 C CNN
-F 1 "10k" V 2800 6800 50  0000 C CNN
-F 2 "Resistor_SMD:R_0805_2012Metric_Pad1.20x1.40mm_HandSolder" V 2930 6800 50  0001 C CNN
-F 3 "~" H 3000 6800 50  0001 C CNN
-	1    3000 6800
-	0    -1   -1   0
-$EndComp
-$Comp
 L power:+3V3 #PWR0159
 U 1 1 60256D6F
@@
 Wire Wire Line
 	3350 6700 3350 6800
-Wire Wire Line
-	3350 6800 3150 6800
-Wire Wire Line
-	2850 6800 2750 6800
 Wire Wire Line
 	1700 6850 1750 6850
@@
 Wire Wire Line
 	21300 13600 21300 13800
+$Comp
+L Device:R R15
+U 1 1 60130731
+P 3000 6800
+F 0 "R15" V 2900 6800 50  0000 C CNN
+F 1 "10k" V 2800 6800 50  0000 C CNN
+F 2 "Resistor_SMD:R_0805_2012Metric_Pad1.20x1.40mm_HandSolder" V 2930 6800 50  0001 C CNN
+F 3 "~" H 3000 6800 50  0001 C CNN
+	1    3000 6800
+	0    1    1    0
+$EndComp
+Wire Wire Line
+	3150 6800 3350 6800
+Wire Wire Line
+	2750 6800 2850 6800
+$Comp
+L sch-lib:A25L032 U2
+U 1 1 60070B82
+P 2250 6750
+F 0 "U2" H 1900 7250 50  0000 C CNN
+F 1 "A25L032" H 2000 7150 50  0000 C CNN
+F 2 "TinXsat:WSON-8-1EP_6x5mm_P1.27mm_EP3.4x4mm" H 2250 6150 50  0001 C CNN
+F 3 "http://www.elm-tech.com/en/products/spi-flash-memory/gd25d10/gd25d10.pdf" H 2250 6750 50  0001 C CNN
+	1    2250 6750
+	1    0    0    -1
+$EndComp
 $EndSCHEMATC

Commit message: pcb final commit after chinese changes
Connections:
- net +3.3VP is gone; now on net +3V3: R1.2
Other:
- moved on the sheet: J7, XS1
Changed lines of the file:
@@
 	4700 12350 4700 12650
 Connection ~ 4700 12650
-$Comp
-L power:+3.3VP #PWR0201
-U 1 1 61CD4E41
-P 3750 13150
-F 0 "#PWR0201" H 3900 13100 50  0001 C CNN
-F 1 "+3.3VP" H 3765 13323 50  0000 C CNN
-F 2 "" H 3750 13150 50  0001 C CNN
-F 3 "" H 3750 13150 50  0001 C CNN
-	1    3750 13150
-	1    0    0    -1
-$EndComp
 Wire Wire Line
 	4150 13200 4200 13200
@@
 F 0 "U4" H 7050 3393 60  0000 C CNN
 F 1 "TP4056" H 7050 3287 60  0000 C CNN
-F 2 "Package_SO:SOIC-8-1EP_3.9x4.9mm_P1.27mm_EP2.29x3mm" H 7050 3181 60  0000 C CNN
+F 2 "Package_SO:SOIC-8-1EP_3.9x4.9mm_P1.27mm_EP2.29x3mm" H 7050 3181 60  0001 C CNN
 F 3 "" H 7050 2750 60  0000 C CNN
 	1    7050 2750
@@
 	20900 11900 21550 11900
 $Comp
-L uSD_push-push_ebay:SD_ebay-uSD-push_push_SMD XS1
-U 1 1 61BF60BB
-P 4600 3950
-F 0 "XS1" H 4296 3996 50  0000 R CNN
-F 1 "SD_ebay-uSD-push_push_SMD" H 4296 3905 50  0000 R CNN
-F 2 "footprints:Conn_uSDcard" H 4600 3950 10  0001 C CNN
-F 3 "_" H 4600 3950 10  0001 C CNN
-F 4 "_" H 4600 3950 10  0001 C CNN "Manf#"
-F 5 "ebay" H 4600 3950 10  0001 C CNN "Manf"
-	1    4600 3950
-	1    0    0    -1
-$EndComp
-$Comp
 L Analog_ADC:INA219AxDCN U7
 U 1 1 6237EB1E
@@
 L Connector:Conn_01x09_Female J7
 U 1 1 5FEDD748
-P 5700 3850
-F 0 "J7" H 5728 3876 50  0000 L CNN
-F 1 "ESP-card" H 5728 3785 50  0000 L CNN
-F 2 "TinXsat:PinHeader_1x08_P2mm_SMD" H 5700 3850 50  0001 C CNN
-F 3 "~" H 5700 3850 50  0001 C CNN
-	1    5700 3850
-	1    0    0    -1
-$EndComp
-Wire Wire Line
-	5200 3450 5200 3850
-Wire Wire Line
-	5200 3850 5000 3850
-Wire Wire Line
-	5200 3450 5500 3450
-Wire Wire Line
-	5500 3550 5250 3550
-Wire Wire Line
-	5250 3550 5250 3700
-Wire Wire Line
-	5250 3700 5000 3700
-Wire Wire Line
-	5000 3550 5150 3550
-Wire Wire Line
-	5150 3550 5150 3650
-Wire Wire Line
-	5150 3650 5500 3650
-Wire Wire Line
-	4450 3250 4450 3200
-Wire Wire Line
-	4450 3200 5300 3200
-Wire Wire Line
-	5300 3200 5300 3750
-Wire Wire Line
-	5300 3750 5500 3750
-Wire Wire Line
-	5500 3850 5350 3850
-Wire Wire Line
-	5350 3850 5350 3400
-Wire Wire Line
-	5350 3400 5000 3400
-Wire Wire Line
-	4450 4450 4450 4500
-Wire Wire Line
-	4450 4500 5100 4500
-Wire Wire Line
-	5100 4500 5100 3950
-Wire Wire Line
-	5100 3950 5500 3950
-Wire Wire Line
-	5500 4050 5150 4050
-Wire Wire Line
-	5150 4050 5150 4150
-Wire Wire Line
-	5150 4150 5000 4150
-Wire Wire Line
-	5000 4000 5250 4000
-Wire Wire Line
-	5250 4000 5250 4150
-Wire Wire Line
-	5250 4150 5500 4150
-Wire Wire Line
-	5500 4250 5150 4250
-Wire Wire Line
-	5150 4250 5150 4300
-Wire Wire Line
-	5150 4300 5000 4300
+P 2900 14300
+F 0 "J7" H 2928 14326 50  0000 L CNN
+F 1 "ESP-card" H 2928 14235 50  0000 L CNN
+F 2 "TinXsat:PinHeader_1x08_P2mm_SMD" H 2900 14300 50  0001 C CNN
+F 3 "~" H 2900 14300 50  0001 C CNN
+	1    2900 14300
+	1    0    0    -1
+$EndComp
+Wire Wire Line
+	2400 13900 2400 14300
+Wire Wire Line
+	2400 14300 2200 14300
+Wire Wire Line
+	2400 13900 2700 13900
+Wire Wire Line
+	2700 14000 2450 14000
+Wire Wire Line
+	2450 14000 2450 14150
+Wire Wire Line
+	2450 14150 2200 14150
+Wire Wire Line
+	2200 14000 2350 14000
+Wire Wire Line
+	2350 14000 2350 14100
+Wire Wire Line
+	2350 14100 2700 14100
+Wire Wire Line
+	1650 13700 1650 13650
+Wire Wire Line
+	1650 13650 2500 13650
+Wire Wire Line
+	2500 13650 2500 14200
+Wire Wire Line
+	2500 14200 2700 14200
+Wire Wire Line
+	2700 14300 2550 14300
+Wire Wire Line
+	2550 14300 2550 13850
+Wire Wire Line
+	2550 13850 2200 13850
+Wire Wire Line
+	1650 14900 1650 14950
+Wire Wire Line
+	1650 14950 2300 14950
+Wire Wire Line
+	2300 14950 2300 14400
+Wire Wire Line
+	2300 14400 2700 14400
+Wire Wire Line
+	2700 14500 2350 14500
+Wire Wire Line
+	2350 14500 2350 14600
+Wire Wire Line
+	2350 14600 2200 14600
+Wire Wire Line
+	2200 14450 2450 14450
+Wire Wire Line
+	2450 14450 2450 14600
+Wire Wire Line
+	2450 14600 2700 14600
+Wire Wire Line
+	2700 14700 2350 14700
+Wire Wire Line
+	2350 14700 2350 14750
+Wire Wire Line
+	2350 14750 2200 14750
 Text GLabel 1700 6850 0    50   Input ~ 0
 FLASH_WP
@@
 L power:GND #PWR0219
 U 1 1 5FF2DAEA
-P 5100 4500
-F 0 "#PWR0219" H 5100 4250 50  0001 C CNN
-F 1 "GND" H 5105 4327 50  0000 C CNN
-F 2 "" H 5100 4500 50  0001 C CNN
-F 3 "" H 5100 4500 50  0001 C CNN
-	1    5100 4500
-	1    0    0    -1
-$EndComp
-Connection ~ 5100 4500
+P 2300 14950
+F 0 "#PWR0219" H 2300 14700 50  0001 C CNN
+F 1 "GND" H 2305 14777 50  0000 C CNN
+F 2 "" H 2300 14950 50  0001 C CNN
+F 3 "" H 2300 14950 50  0001 C CNN
+	1    2300 14950
+	1    0    0    -1
+$EndComp
+Connection ~ 2300 14950
 $Comp
 L power:VDD #PWR0128
@@
 	1    0    0    -1
 $EndComp
+$Comp
+L uSD_push-push_ebay:SD_ebay-uSD-push_push_SMD XS1
+U 1 1 61BF60BB
+P 1800 14400
+F 0 "XS1" H 1496 14446 50  0000 R CNN
+F 1 "SD_ebay-uSD-push_push_SMD" H 1496 14355 50  0000 R CNN
+F 2 "footprints:Conn_uSDcard" H 1800 14400 10  0001 C CNN
+F 3 "_" H 1800 14400 10  0001 C CNN
+F 4 "_" H 1800 14400 10  0001 C CNN "Manf#"
+F 5 "ebay" H 1800 14400 10  0001 C CNN "Manf"
+	1    1800 14400
+	1    0    0    -1
+$EndComp
+$Comp
+L power:+3V3 #PWR?
+U 1 1 5FF40037
+P 3750 13150
+F 0 "#PWR?" H 3750 13000 50  0001 C CNN
+F 1 "+3V3" H 3765 13323 50  0000 C CNN
+F 2 "" H 3750 13150 50  0001 C CNN
+F 3 "" H 3750 13150 50  0001 C CNN
+	1    3750 13150
+	1    0    0    -1
+$EndComp
